File: hw/mainBoard.kicad_pcb (KiCad board)
At the start: 2 copper layers, 63.5 x 53.3 mm, 67 parts, among them J1 Y, J2 X, J3 PWR_5, J4 LASER, J5 PWR_15, J6 FTDI, Q1 BC817, Q2 BC817, U1 DAC8562, U2 AP1117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

Commit message: Final touch on the board
Routing:
- net GND: track 132.4 -> 105.8 mm, vias 13 -> 15
- net -15V: track 46.6 -> 52.0 mm, vias 1 -> 0
- net SCK: track 28.9 -> 29.7 mm
- net SYNC: track 25.1 -> 26.0 mm
- net DATA: track 32.0 -> 32.8 mm
- net CLR: track 34.6 -> 35.5 mm
- net LDAC: track 33.4 -> 34.2 mm
- net +5V: track 69.8 -> 70.5 mm
- net BOOT: track 14.8 -> 15.5 mm
- net +9VA: track 86.4 -> 87.1 mm
- net LASER: track 69.1 -> 69.8 mm
- net -9VA: track 67.3 -> 67.9 mm, vias 2 -> 4
- added copper zone on F.Cu, net GND
Other:
- board text added: "LaserProjector v1.0 Jan Mrázek 8/2017 honzamrazek.cz"
